Commit message: 2.5,5

File: install/smart_car/share/smart_car/urdf/smartcar.urdf.xacro (robot description, xacro)
@@ -1,214 +1 @@
-<?xml version="1.0"?>
-<robot name="mobile_robot" xmlns:xacro="http://www.ros.org/wiki/xacro">
-  <xacro:property name="PI" value="3.1415926535897931"/>
-  <xacro:property name="wheel_diameter" value="0.064"/>
-  <xacro:property name="wheel_radius" value="${wheel_diameter/2}"/>
-  <xacro:property name="wheel_width" value="0.025"/>
-  <xacro:property name="wheelbase_length" value="0.257"/>
-  <xacro:property name="wheelbase_width" value="0.17"/>
-  <xacro:property name="chassis_height" value="0.05"/>
-  <xacro:property name="chassis_mass" value="5.0"/>
-  <xacro:property name="wheel_mass" value="0.1"/>
-  <xacro:property name="steer_link_mass" value="0.05"/>
-  <!-- Inertia macros -->
-  <xacro:macro name="box_inertia" params="m x y z">
-    <inertial>
-      <mass value="${m}"/>
-      <inertia ixx="${(1/12) * m * (y*y + z*z)}" ixy="0.0" ixz="0.0"
-               iyy="${(1/12) * m * (x*x + z*z)}" iyz="0.0"
-               izz="${(1/12) * m * (x*x + y*y)}"/>
-    </inertial>
-  </xacro:macro>
-  <xacro:macro name="cylinder_inertia" params="m r h">
-    <inertial>
-      <mass value="${m}"/>
-      <inertia ixx="${(1/12) * m * (3*r*r + h*h)}" ixy="0.0" ixz="0.0"
-               iyy="${(1/2) * m * r*r}" iyz="0.0"
-               izz="${(1/12) * m * (3*r*r + h*h)}"/>
-    </inertial>
-  </xacro:macro>
-  <!-- Base link -->
-  <link name="base_footprint"/>
-  <joint name="chassis_joint" type="fixed">
-    <parent link="base_footprint"/>
-    <child link="Chassis_link"/>
-    <origin xyz="0 0 ${wheel_radius}" rpy="0 0 0"/>
-  </joint>
-  <link name="Chassis_link">
-    <visual>
-      <geometry>
-        <box size="${wheelbase_length} ${wheelbase_width} ${chassis_height}"/>
-      </geometry>
-      <material name="grey">
-        <color rgba="0.5 0.5 0.5 1.0"/>
-      </material>
-    </visual>
-    <collision>
-      <geometry>
-        <box size="${wheelbase_length} ${wheelbase_width} ${chassis_height}"/>
-      </geometry>
-    </collision>
-    <xacro:box_inertia m="${chassis_mass}" x="${wheelbase_length}" y="${wheelbase_width}" z="${chassis_height}"/>
-  </link>
-  <joint name="base_link_joint" type="fixed">
-    <parent link="Chassis_link"/>
-    <child link="base_link"/>
-    <origin xyz="0 0 0" rpy="0 0 0"/>
-  </joint>
-  <link name="base_link"/>
-  <!-- Wheels -->
-  <xacro:macro name="wheel" params="prefix side reflect">
-    <link name="${prefix}_${side}_wheel_link">
-      <visual>
-        <origin xyz="0 0 0" rpy="${PI/2} 0 0"/>
-        <geometry>
-          <cylinder radius="${wheel_radius}" length="${wheel_width}"/>
-        </geometry>
-        <material name="black">
-          <color rgba="0.1 0.1 0.1 1.0"/>
-        </material>
-      </visual>
-      <collision>
-        <origin xyz="0 0 0" rpy="${PI/2} 0 0"/>
-        <geometry>
-          <cylinder radius="${wheel_radius}" length="${wheel_width}"/>
-        </geometry>
-      </collision>
-      <xacro:cylinder_inertia m="${wheel_mass}" r="${wheel_radius}" h="${wheel_width}"/>
-    </link>
-  </xacro:macro>
-  <xacro:wheel prefix="back" side="left" reflect="1"/>
-  <xacro:wheel prefix="back" side="right" reflect="-1"/>
-  <joint name="back_left_wheel_joint" type="continuous">
-    <parent link="Chassis_link"/>
-    <child link="back_left_wheel_link"/>
-    <origin xyz="-${wheelbase_length/2} ${wheelbase_width/2} 0" rpy="0 0 0"/>
-    <axis xyz="0 1 0"/>
-  </joint>
-  <joint name="back_right_wheel_joint" type="continuous">
-    <parent link="Chassis_link"/>
-    <child link="back_right_wheel_link"/>
-    <origin xyz="-${wheelbase_length/2} -${wheelbase_width/2} 0" rpy="0 0 0"/>
-    <axis xyz="0 1 0"/>
-  </joint>
-  <xacro:wheel prefix="front" side="left" reflect="1"/>
-  <xacro:wheel prefix="front" side="right" reflect="-1"/>
-  <joint name="front_right_wheel_steer_joint" type="revolute">
-    <parent link="Chassis_link"/>
-    <child link="front_right_steer_link"/>
-    <origin xyz="${wheelbase_length/2} -${wheelbase_width/2} 0"/>
-    <axis xyz="0 0 1"/>
-    <limit lower="-0.6" upper="0.6" effort="10" velocity="100"/>
-  </joint>
-  <link name="front_right_steer_link">
-    <xacro:box_inertia m="${steer_link_mass}" x="0.01" y="0.01" z="0.01"/>
-  </link>
-  <joint name="front_right_wheel_joint" type="continuous">
-    <parent link="front_right_steer_link"/>
-    <child link="front_right_wheel_link"/>
-    <origin xyz="0 0 0"/>
-    <axis xyz="0 1 0"/>
-  </joint>
-  <joint name="front_left_wheel_steer_joint" type="revolute">
-    <parent link="Chassis_link"/>
-    <child link="front_left_steer_link"/>
-    <origin xyz="${wheelbase_length/2} ${wheelbase_width/2} 0"/>
-    <axis xyz="0 0 1"/>
-    <limit lower="-0.6" upper="0.6" effort="10" velocity="100"/>
-  </joint>
-  <link name="front_left_steer_link">
-     <xacro:box_inertia m="${steer_link_mass}" x="0.01" y="0.01" z="0.01"/>
-  </link>
-  <joint name="front_left_wheel_joint" type="continuous">
-    <parent link="front_left_steer_link"/>
-    <child link="front_left_wheel_link"/>
-    <origin xyz="0 0 0"/>
-    <axis xyz="0 1 0"/>
-  </joint>
-  <!-- ==================== IMU SENSOR ==================== -->
-  <!-- Add IMU link & mount BEFORE sensor definition -->
-  <link name="imu_link">
-    <inertial>
-      <mass value="0.01"/>
-      <inertia ixx="1e-6" iyy="1e-6" izz="1e-6" ixy="0" ixz="0" iyz="0"/>
-    </inertial>
-  </link>
-  <joint name="imu_mount" type="fixed">
-    <parent link="base_link"/>
-    <child link="imu_link"/>
-    <origin xyz="0 0 ${chassis_height + 0.03}" rpy="0 0 0"/>
-  </joint>
-  <gazebo reference="imu_link">
-    <sensor name="imu_sensor" type="imu">
-      <always_on>true</always_on>
-      <update_rate>100.0</update_rate>
-      <imu>
-        <noise>
-          <!-- noise parameters kept -->
-        </noise>
-      </imu>
-      <plugin name="imu_plugin" filename="libgazebo_ros_imu_sensor.so">
-        <ros>
-          <namespace>/</namespace>
-          <remapping>/imu_plugin/out:=/imu_data</remapping>
-        </ros>
-      </plugin>
-    </sensor>
-  </gazebo>
-  <!-- ==================== LIDAR SENSOR ==================== -->
-  <link name="sllidar_base_link">
-    <visual>
-      <geometry>
-        <cylinder radius="0.04" length="0.05"/>
-      </geometry>
-      <material name="red">
-        <color rgba="1 0 0 1"/>
-      </material>
-    </visual>
-  </link>
-  <joint name="lidar_joint" type="fixed">
-    <parent link="base_link"/>
-    <child link="sllidar_base_link"/>
-    <origin xyz="${wheelbase_length/2} 0 ${chassis_height + 0.05}" rpy="0 0 0"/>
-  </joint>
-  <gazebo reference="sllidar_base_link">
-    <sensor name="lidar_sensor" type="ray">
-      <pose>0 0 0 0 0 0</pose>
-      <visualize>true</visualize>
-      <update_rate>20.0</update_rate>
-      <ray>
-        <scan>
-          <horizontal>
-            <samples>200</samples>
-            <resolution>1</resolution>
-            <min_angle>-0.7854</min_angle>
-            <max_angle>0.7854</max_angle>
-          </horizontal>
-        </scan>
-        <range>
-          <min>0.12</min>
-          <max>6.0</max>
-          <resolution>0.01</resolution>
-        </range>
-        <noise>
-          <type>gaussian</type>
-          <mean>0.0</mean>
-          <stddev>0.01</stddev>
-        </noise>
-      </ray>
-      <plugin name="gazebo_ros_laser" filename="libgazebo_ros_ray_sensor.so">
-        <ros>
-          <namespace>/</namespace>
-          <remapping>/gazebo_ros_laser/out:=/scan</remapping>
-        </ros>
-        <output_type>sensor_msgs/LaserScan</output_type>
-        <frame_name>sllidar_base_link</frame_name>
-      </plugin>
-    </sensor>
-  </gazebo>
-  <!-- VEHICLE CONTROL PLUGIN OUTSIDE SENSOR -->
-  <gazebo>
-    <plugin name="car_gazebo_plugin" filename="libcar_gazebo_plugin.so">
-    </plugin>
-  </gazebo>
-</robot>
+/home/yappel/ros2_ws/src/smart_car/urdf/smartcar.urdf.xacro
